File: _autosave-Custom_devboard.kicad_pcb (KiCad board)
At the start: 2 copper layers, 21 x 51 mm, 33 parts, among them J1 USB_C_Receptacle_USB2.0_14P, J2 Conn_01x20, J3 Conn_01x20, J4 Conn_01x03, SW1 SW_Push, U1 RP2040, U2 MCP1700x-330xxTT, U3 W25Q128JVS, U4 W25Q16JVZPIQ TR, Y1 12 MHz

Commit message: Working on PCB (just placing everyhting)
Parts:
- removed U3: W25Q128JVS, Package_SO:SOIC-8_5.3x5.3mm_P1.27mm
- moved U4 228.4 mm to (210.6, 94.8)
- moved R4 184.0 mm to (214.1, 97.5), turned to -90 degrees
- moved C15 168.0 mm to (215.0, 111.5), turned to 90 degrees
- moved U2 165.8 mm to (210.5, 83.5), turned to 90 degrees
- moved Y1 163.0 mm to (212.5, 111.5)
- moved C16 162.7 mm to (210.0, 111.5), turned to -90 degrees
- moved C14 141.4 mm to (186.2, 113.0)
- moved C1 136.9 mm to (173.5, 73.7)
- moved C10 136.9 mm to (176.4, 79.6)
- moved C11 136.9 mm to (176.4, 81.6)
- moved C12 136.9 mm to (180.1, 113.2)
- moved C13 136.9 mm to (180.1, 115.0)
- moved C2 136.9 mm to (173.5, 75.7)
- moved C3 136.9 mm to (173.5, 77.6)
- moved C4 136.9 mm to (173.5, 79.6)
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Routing:
- net QSPI_SS: track 0.00 -> 7.55 mm
- net QSPI_SD1: track 0.00 -> 6.85 mm
- net QSPI_SD3: track 0.00 -> 6.24 mm
- net QSPI_SD2: track 0.00 -> 5.89 mm
- net QSPI_SCLK: track 0.00 -> 5.46 mm
- net QSPI_SD0: track 0.00 -> 4.10 mm
- net USBD-: track 0.00 -> 3.11 mm
- net USBD+: track 0.00 -> 2.99 mm

Commit message: PCB, CONECTING EVERYHTING SUCKS SO BAD
Parts:
- moved R5 54.6 mm to (216.4, 111.3)
- moved C4 52.1 mm to (219.6, 104.0)
- moved C2 51.4 mm to (219.0, 99.5)
- moved C10 50.2 mm to (217.0, 109.2), turned to 180 degrees
- moved R3 48.8 mm to (215.2, 97.5), turned to -90 degrees
- moved C5 48.2 mm to (213.5, 108.5), turned to -90 degrees
- moved C11 47.5 mm to (215.1, 109.0)
- moved C9 47.3 mm to (219.0, 98.0)
- moved C8 46.6 mm to (217.5, 97.5), turned to 90 degrees
- moved R2 45.9 mm to (214.5, 89.0), turned to -90 degrees
- moved R1 45.9 mm to (215.5, 83.0), turned to 180 degrees
- moved C13 44.0 mm to (208.5, 81.5), turned to 180 degrees
- moved C1 43.7 mm to (208.0, 100.5), turned to 180 degrees
- moved C3 43.4 mm to (208.0, 104.0), turned to 180 degrees
- moved C7 42.5 mm to (217.5, 84.5), turned to 180 degrees
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Routing:
- net GND: track 0.00 -> 169.0 mm, vias 0 -> 3
- net +3V3: track 0.00 -> 40.0 mm
- net GPIO15: track 0.00 -> 19.8 mm
- net USBD+: track 2.99 -> 21.8 mm
- net USBD-: track 3.11 -> 21.7 mm
- net GPIO14: track 0.00 -> 18.0 mm
- net VBUS: track 0.00 -> 13.0 mm
- net +1V1: track 0.00 -> 12.7 mm
- net GPIO13: track 0.00 -> 11.8 mm
- net GPIO24: track 0.00 -> 10.2 mm
- net Net-(J1-CC2): track 0.00 -> 10.2 mm
- net GPIO12: track 0.00 -> 9.14 mm
- net XIN: track 0.00 -> 8.77 mm
- net GPIO11: track 0.00 -> 7.45 mm
- net GPIO10: track 0.00 -> 6.57 mm
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