File: _autosave-Custom_devboard.kicad_pcb (KiCad board)
At the start: 2 copper layers, 21 x 51 mm, 32 parts, among them J1 USB_C_Receptacle_USB2.0_14P, J2 Conn_01x20, J3 Conn_01x20, J4 Conn_01x03, SW1 SW_Push, U1 RP2040, U2 MCP1700x-330xxTT, U4 W25Q16JVZPIQ TR, Y1 12 MHz

Commit message: GND and DRC
Parts:
- moved C15 0.06 mm to (152.0, 123.2)
Routing:
- net GND: track 33.7 -> 97.4 mm, vias 0 -> 18
- net +3V3: track 61.2 -> 77.9 mm, vias 4 -> 7
- net (no net): track 6.34 -> 0.00 mm
- net SWCLK: track 18.2 -> 20.1 mm
- net GPIO26/ADC0: track 15.6 -> 17.3 mm
- net SWD: track 16.9 -> 18.6 mm
- net +1V1: track 25.9 -> 27.6 mm
- net Net-(C15-Pad2): track 3.65 -> 4.23 mm
- added copper zone on B.Cu, net GND
- added copper zone on F.Cu, net GND
