File: Custom_devboard.kicad_pcb (KiCad board)
At the start: 2 copper layers, 21 x 51 mm, 32 parts, among them J1 USB_C_Receptacle_USB2.0_14P, J2 Conn_01x20, J3 Conn_01x20, J4 Conn_01x03, SW1 SW_Push, U1 RP2040, U2 MCP1700x-330xxTT, U4 W25Q16JVZPIQ TR, Y1 12 MHz

Commit message: SilkScreen is done
Parts:
- C3: moved to F.Cu
- moved R5 67.6 mm to (149.4, 120.2), turned to 90 degrees
- moved R2 66.0 mm to (148.7, 93.6)
- moved C10 65.6 mm to (152.6, 121.9), turned to 0 degrees
- moved C3 64.6 mm to (144.6, 116.3), turned to 180 degrees
- moved U2 64.2 mm to (147.4, 95.8)
- moved C12 64.1 mm to (153.0, 109.3)
- moved C14 64.1 mm to (147.4, 98.2)
- moved C16 64.1 mm to (146.9, 123.2)
- moved C2 64.1 mm to (155.9, 111.2)
- moved C4 64.1 mm to (156.5, 115.7)
- moved C5 64.1 mm to (150.5, 120.2)
- moved C6 64.1 mm to (148.4, 104.7)
- moved C8 64.1 mm to (154.4, 109.1)
- moved C9 64.1 mm to (155.9, 109.7)
- moved J2 64.1 mm to (141.6, 86.5)
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Routing:
- net GND: track 173.4 -> 97.4 mm, vias 3 -> 19
- net +3V3: track 42.0 -> 77.9 mm, vias 0 -> 7
- net GPIO0: track 0.00 -> 28.7 mm, vias 0 -> 1
- net GPIO1: track 0.00 -> 27.4 mm, vias 0 -> 1
- net GPIO29/ADC3: track 0.00 -> 27.0 mm, vias 0 -> 1
- net GPIO2: track 0.00 -> 22.5 mm, vias 0 -> 1
- net GPIO28/ADC2: track 0.00 -> 21.6 mm, vias 0 -> 1
- net GPIO3: track 0.00 -> 20.7 mm
- net GPIO4: track 0.00 -> 19.4 mm
- net GPIO5: track 0.00 -> 18.7 mm
- net GPIO27/ADC1: track 0.00 -> 17.6 mm, vias 0 -> 1
- net GPIO26/ADC0: track 0.00 -> 17.3 mm
- net +1V1: track 13.4 -> 27.6 mm, vias 0 -> 2
- net GPIO6: track 0.00 -> 12.9 mm
- net GPIO7: track 0.00 -> 11.3 mm
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- added copper zone on B.Cu, net GND
- added copper zone on F.Cu, net GND
Other:
- board text added: "Sana Deghat!!"

Commit message: final btw
Parts:
- added G***: LOGO, LOGO, B.Cu at (153.1, 97.8)
- added G***: LOGO, LOGO, B.Cu at (147.7, 125.7)
Other:
- board text added: "Socretes"
