File: Custom_devboard.kicad_sch (KiCad schematic)
At the start: 0 parts

Commit message: Designing the schematic for the devboard
Parts:
- added C1, C11, C12, C2, C3, C4, C6, C7, C8, C9: 0.1uf, symbol Device:C
- added C10, C5: 1uf, symbol Device:C
- added C13, C14: 10uf, symbol Device:C
- added C15, C16: 15pF, symbol Device:C
- added J1: USB_C_Receptacle_USB2.0_14P, symbol Connector:USB_C_Receptacle_USB2.0_14P
- added J2, J3: Conn_01x20, symbol Connector_Generic:Conn_01x20
- added J4: Conn_01x03, symbol Connector_Generic:Conn_01x03
- added R1, R2: 5.1k, symbol Device:R
- added R3, R4: 27, symbol Device:R
- added R5, R7: 1k, symbol Device:R
- added R6: 10k, symbol Device:R
- added SW1: SW_Push, symbol Switch:SW_Push
- added U1: RP2040, Package_DFN_QFN:QFN-56-1EP_7x7mm_P0.4mm_EP3.2x3.2mm, symbol MCU_RaspberryPi:RP2040
- added U2: NCP1117-3.3_SOT223, Package_TO_SOT_SMD:SOT-223-3_TabPin2, symbol Regulator_Linear:NCP1117-3.3_SOT223
- added U3: W25Q128JVS, Package_SO:SOIC-8_5.3x5.3mm_P1.27mm, symbol Memory_Flash:W25Q128JVS
- added Y1: 12 MHz, symbol Device:Crystal_GND24
Connections:
- new net: C15.2, R5.1, Y1.3
- new net: R3.2, U1.46 (USB_DM)
- new net: J1.B5 (CC2), R2.1
- new net: R7.1, SW1.2
- new net: R4.2, U1.47 (USB_DP)
- new net: J1.A5 (CC1), R1.2
- new net +1V1: C10.1, C11.1, C12.1, U1.23 (DVDD), U1.45 (VREG_VOUT), U1.50 (DVDD)
- new net +3V3: C1.1, C14.1, C2.1, C3.1, C4.1, C5.1, C6.1, C7.1, C8.1, C9.1, J3.5 (Pin_5), R6.1, U1.1 (IOVDD), U1.10 (IOVDD), U1.22 (IOVDD), U1.33 (IOVDD), U1.42 (IOVDD), U1.43 (ADC_AVDD), U1.44 (VREG_VIN), U1.48 (USB_VDD), U1.49 (IOVDD), U2.2 (VO), U3.8 (VCC)
- new net GND: C1.2, C10.2, C11.2, C12.2, C13.2, C14.2, C15.1, C16.1, C2.2, C3.2, C4.2, C5.2, C6.2, C7.2, C8.2, C9.2, J1.A1 (GND), J1.A12 (GND), J1.B1 (GND), J1.B12 (GND), J1.S1 (SHIELD), J2.13 (Pin_13), J2.18 (Pin_18), J2.3 (Pin_3), J2.8 (Pin_8), J3.13 (Pin_13), J3.18 (Pin_18), J3.3 (Pin_3), J3.8 (Pin_8), J4.2 (Pin_2), R1.1, R2.2, SW1.1, U2.1 (GND), U3.4 (GND), Y1.2 (G), Y1.4 (G)
- new net GPIO0: J2.1 (Pin_1), U1.2 (GPIO0)
- new net GPIO1: J2.2 (Pin_2), U1.3 (GPIO1)
- new net GPIO10: J2.14 (Pin_14), U1.13 (GPIO10)
- new net GPIO11: J2.15 (Pin_15), U1.14 (GPIO11)
- new net GPIO12: J2.16 (Pin_16), U1.15 (GPIO12)
- new net GPIO13: J2.17 (Pin_17), U1.16 (GPIO13)
- new net GPIO14: J2.19 (Pin_19), U1.17 (GPIO14)
- new net GPIO15: J2.20 (Pin_20), U1.18 (GPIO15)
- new net GPIO16: J3.20 (Pin_20), U1.27 (GPIO16)
- new net GPIO17: J3.19 (Pin_19), U1.28 (GPIO17)
- new net GPIO18: J3.17 (Pin_17), U1.29 (GPIO18)
- new net GPIO19: J3.16 (Pin_16), U1.30 (GPIO19)
- new net GPIO2: J2.4 (Pin_4), U1.4 (GPIO2)
- new net GPIO20: J3.15 (Pin_15), U1.31 (GPIO20)
- new net GPIO21: J3.14 (Pin_14), U1.32 (GPIO21)
- new net GPIO22: J3.12 (Pin_12), U1.34 (GPIO22)
- new net GPIO23: U1.35 (GPIO23)
- new net GPIO24: U1.36 (GPIO24)
- new net GPIO26/ADC0: J3.10 (Pin_10), U1.38 (GPIO26/ADC0)
- new net GPIO27/ADC1: J3.9 (Pin_9), U1.39 (GPIO27/ADC1)
- new net GPIO28/ADC2: J3.7 (Pin_7), U1.40 (GPIO28/ADC2)
- new net GPIO29/ADC3: U1.41 (GPIO29/ADC3)
- new net GPIO3: J2.5 (Pin_5), U1.5 (GPIO3)
- new net GPIO4: J2.6 (Pin_6), U1.6 (GPIO4)
- new net GPIO5: J2.7 (Pin_7), U1.7 (GPIO5)
- new net GPIO6: J2.9 (Pin_9), U1.8 (GPIO6)
- new net GPIO7: J2.10 (Pin_10), U1.9 (GPIO7)
- new net GPIO8: J2.11 (Pin_11), U1.11 (GPIO8)
- new net GPIO9: J2.12 (Pin_12), U1.12 (GPIO9)
- new net QSPI_SCLK: U1.52 (QSPI_SCLK), U3.6 (CLK)
- new net QSPI_SD0: U1.53 (QSPI_SD0), U3.5 (DI/IO_{0})
- new net QSPI_SD1: U1.55 (QSPI_SD1), U3.2 (DO/IO_{1})
- new net QSPI_SD2: U1.54 (QSPI_SD2), U3.3 (~{WP}/IO_{2})
- new net QSPI_SD3: U1.51 (QSPI_SD3), U3.7 (~{HOLD}/~{RESET}/IO_{3})
- new net QSPI_SS: R6.2, R7.2, U1.56 (~{QSPI_SS}), U3.1 (~{CS})
- new net RUN: J3.11 (Pin_11)
- new net SWCLK: J4.1 (Pin_1), U1.24 (SWCLK)
- new net SWD: J4.3 (Pin_3), U1.25 (SWDIO)
- new net USBD+: J1.A6 (D+), J1.B6 (D+), R4.1
- new net USBD-: J1.A7 (D-), J1.B7 (D-), R3.1
- new net VBUS: C13.1, J1.A4 (VBUS), J1.A9 (VBUS), J1.B4 (VBUS), J1.B9 (VBUS), J3.1 (Pin_1), U2.3 (VI)
- new net XIN: C16.2, U1.20 (XIN), Y1.1
- new net XOUT: R5.2, U1.21 (XOUT)
- no-connect marks 0 -> 1

Commit message: footprint complete and ERC
Parts:
- removed U2: NCP1117-3.3_SOT223, Package_TO_SOT_SMD:SOT-223-3_TabPin2, symbol Regulator_Linear:NCP1117-3.3_SOT223
- added U2: MCP1700x-330xxTT, Package_TO_SOT_SMD:SOT-23, symbol Regulator_Linear:MCP1700x-330xxTT
- C1, C10, C11, C2, C3, C4, C5, C6, C7, C8, C9: footprint (none) -> Capacitor_SMD:C_0402_1005Metric
- C12, C13, C14: footprint (none) -> Capacitor_SMD:C_0201_0603Metric
- C15, C16: value 15pF -> 33pF; footprint (none) -> Capacitor_SMD:C_0201_0603Metric
- J1: footprint (none) -> Connector_USB:USB_C_Receptacle_HRO_TYPE-C-31-M-12
- J2, J3: footprint (none) -> Connector_PinHeader_2.54mm:PinHeader_1x20_P2.54mm_Vertical
- J4: footprint (none) -> Connector_PinHeader_2.54mm:PinHeader_1x03_P2.54mm_Vertical
- R1, R2, R3, R4, R5, R6, R7: footprint (none) -> Resistor_SMD:R_0402_1005Metric
- SW1: footprint (none) -> Button_Switch_SMD:SW_Push_SPST_NO_Alps_SKRK
- U4: renamed from U3; value W25Q128JVS -> W25Q16JVZPIQ TR; footprint Package_SO:SOIC-8_5.3x5.3mm_P1.27mm -> Package_SON:Winbond_USON-8-1EP_3x2mm_P0.5mm_EP0.2x1.6mm
- Y1: footprint (none) -> Crystal:Crystal_SMD_3225-4Pin_3.2x2.5mm
Connections:
- net +3V3: now also U2.2 (VO)
- net GND: now also U1.19 (TESTEN), U1.57 (GND), U2.1 (GND)
- net GPIO23: now also J3.10 (Pin_10)
- net GPIO24: now also J3.9 (Pin_9)
- net GPIO26/ADC0: now also J3.7 (Pin_7); no longer J3.10 (Pin_10)
- net GPIO27/ADC1: now also J3.6 (Pin_6); no longer J3.9 (Pin_9)
- net GPIO28/ADC2: now also J3.4 (Pin_4); no longer J3.7 (Pin_7)
- net GPIO29/ADC3: now also J3.2 (Pin_2)
- net RUN: now also U1.26 (RUN)
- net VBUS: now also U2.3 (VI)

Commit message: final btw
Changed lines of the file:
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@@
 		(on_board yes)
 		(dnp no)
-		(fields_autoplaced yes)
 		(property "Reference" "#PWR01"
 			(at 173.99 63.5 0)
@@
 		)
 		(property "Value" "+1V1"
-			(at 173.99 54.61 0)
+			(at 176.022 55.118 0)
 			(effects
 				(font
@@
 		(dnp no)
 		(property "Reference" "U1"
-			(at 169.926 150.368 0)
-			(effects
-				(font
+			(at 170.688 150.368 0)
+			(effects
+				(font
